File: hardware/muon_detector_head/muon_detector_head.kicad_sch (KiCad schematic)
At the start: 17 parts, among them J1 Conn_01x08, U1 TPH2502, U2 LM393

Commit message: feat: added footprints and custom symbols and stuff
Parts:
- C1, C2, C3, C4, C5: footprint (none) -> Capacitor_SMD:C_0805_2012Metric
- J1: footprint (none) -> Connector_PinHeader_2.54mm:PinHeader_1x08_P2.54mm_Vertical
- R1, R2, R3, R4, R5, R6, R7: footprint (none) -> Resistor_SMD:R_0805_2012Metric
- RV1: footprint (none) -> Potentiometer_SMD:Potentiometer_Bourns_3314G_Vertical
- U1: footprint (none) -> Package_SO:SOIC-8_3.9x4.9mm_P1.27mm
- U2: value LM393 -> TLV3502; footprint (none) -> Package_SO:SOIC-8_3.9x4.9mm_P1.27mm; symbol Comparator:LM393 -> Comparator:TLV3502
Other:
- note added: "U2: VOLTAGE-COMPARATOR"
- note removed: "U2: VOLTAGE-COMPARATOR real part is TLV3502 (push-pull, not open-collector)"
Changed lines of the file:
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@@
 		)
 	)
-	(text "U2: VOLTAGE-COMPARATOR\nreal part is TLV3502 \n(push-pull, not open-collector)"
+	(text "U2: VOLTAGE-COMPARATOR"
 		(exclude_from_sim no)
-		(at 243.84 34.544 0)
+		(at 246.126 36.322 0)
 		(effects
 			(font
@@
 			)
 		)
-		(property "Footprint" ""
+		(property "Footprint" "Resistor_SMD:R_0805_2012Metric"
 			(at 61.722 83.82 90)
 			(effects
@@
 			)
 		)
-		(property "Footprint" ""
+		(property "Footprint" "Resistor_SMD:R_0805_2012Metric"
 			(at 36.322 53.34 90)
 			(effects
@@
 			)
 		)
-		(property "Footprint" ""
+		(property "Footprint" "Capacitor_SMD:C_0805_2012Metric"
 			(at 185.1152 137.16 0)
 			(effects
@@
 			)
 		)
-		(property "Footprint" ""
+		(property "Footprint" "Potentiometer_SMD:Potentiometer_Bourns_3314G_Vertical"
 			(at 233.68 62.23 0)
 			(effects
@@
 			)
 		)
-		(property "Footprint" ""
+		(property "Footprint" "Package_SO:SOIC-8_3.9x4.9mm_P1.27mm"
 			(at 125.73 87.63 0)
 			(effects
@@
 	)
 	(symbol
-		(lib_id "Comparator:LM393")
+		(lib_id "Comparator:TLV3502")
 		(at 243.84 90.17 0)
 		(unit 3)
@@
 			)
 		)
-		(property "Value" "LM393"
+		(property "Value" "TLV3502"
 			(at 242.57 91.4399 0)
 			(effects
@@
 			)
 		)
-		(property "Footprint" ""
+		(property "Footprint" "Package_SO:SOIC-8_3.9x4.9mm_P1.27mm"
 			(at 243.84 90.17 0)
 			(effects
@@
 			)
 		)
-		(property "Datasheet" "http://www.ti.com/lit/ds/symlink/lm393.pdf"
-			(at 243.84 90.17 0)
+		(property "Datasheet" "https://www.ti.com/lit/gpn/TLV3502"
+			(at 243.84 83.566 0)
 			(effects
 				(font
@@
 			)
 		)
-		(property "Description" "Low-Power, Low-Offset Voltage, Dual Comparators, DIP-8/SOIC-8/TO-99-8"
-			(at 243.84 90.17 0)
+		(property "Description" "4.5ns Rail-to-Rail Push-Pull Dual Comparator, SOIC-8"
+			(at 243.332 79.502 0)
 			(effects
 				(font
@@
 			)
 		)
-		(property "Footprint" ""
+		(property "Footprint" "Capacitor_SMD:C_0805_2012Metric"
 			(at 141.9352 137.16 0)
 			(effects
@@
 			)
 		)
-		(property "Footprint" ""
+		(property "Footprint" "Package_SO:SOIC-8_3.9x4.9mm_P1.27mm"
 			(at 186.69 46.99 0)
 			(effects
@@
 			)
 		)
-		(property "Footprint" ""
+		(property "Footprint" "Resistor_SMD:R_0805_2012Metric"
 			(at 261.62 47.752 90)
 			(effects
@@
 			)
 		)
-		(property "Footprint" ""
+		(property "Footprint" "Resistor_SMD:R_0805_2012Metric"
 			(at 185.42 21.082 90)
 			(effects
@@
 			)
 		)
-		(property "Footprint" ""
+		(property "Footprint" "Resistor_SMD:R_0805_2012Metric"
 			(at 94.742 50.8 90)
 			(effects
@@
 			)
 		)
-		(property "Footprint" ""
+		(property "Footprint" "Resistor_SMD:R_0805_2012Metric"
 			(at 159.512 73.66 90)
 			(effects
@@
 	)
 	(symbol
-		(lib_id "Comparator:LM393")
+		(lib_id "Comparator:TLV3502")
 		(at 246.38 49.53 0)
 		(unit 1)
@@
 			)
 		)
-		(property "Value" "LM393"
+		(property "Value" "TLV3502"
 			(at 246.38 41.91 0)
 			(effects
@@
 			)
 		)
-		(property "Footprint" ""
+		(property "Footprint" "Package_SO:SOIC-8_3.9x4.9mm_P1.27mm"
 			(at 246.38 49.53 0)
 			(effects
@@
 			)
 		)
-		(property "Datasheet" "http://www.ti.com/lit/ds/symlink/lm393.pdf"
-			(at 246.38 49.53 0)
+		(property "Datasheet" "https://www.ti.com/lit/gpn/TLV3502"
+			(at 246.38 42.926 0)
 			(effects
 				(font
@@
 			)
 		)
-		(property "Description" "Low-Power, Low-Offset Voltage, Dual Comparators, DIP-8/SOIC-8/TO-99-8"
-			(at 246.38 49.53 0)
+		(property "Description" "4.5ns Rail-to-Rail Push-Pull Dual Comparator, SOIC-8"
+			(at 245.872 38.862 0)
 			(effects
 				(font
@@
 			)
 		)
-		(property "Footprint" ""
+		(property "Footprint" "Resistor_SMD:R_0805_2012Metric"
 			(at 61.722 68.58 90)
 			(effects
@@
 			)
 		)
-		(property "Footprint" ""
+		(property "Footprint" "Capacitor_SMD:C_0805_2012Metric"
 			(at 86.36 43.4848 0)
 			(effects
@@
 			)
 		)
-		(property "Footprint" ""
+		(property "Footprint" "Capacitor_SMD:C_0805_2012Metric"
 			(at 157.1752 137.16 0)
 			(effects
@@
 			)
 		)
-		(property "Footprint" ""
+		(property "Footprint" "Capacitor_SMD:C_0805_2012Metric"
 			(at 171.1452 137.16 0)
 			(effects
@@
 			)
 		)
-		(property "Footprint" ""
+		(property "Footprint" "Package_SO:SOIC-8_3.9x4.9mm_P1.27mm"
 			(at 107.95 78.74 0)
 			(effects
@@
 	)
 	(symbol
-		(lib_id "Comparator:LM393")
+		(lib_id "Comparator:TLV3502")
 		(at 254 113.03 0)
 		(unit 2)
@@
 			)
 		)
-		(property "Value" "LM393"
+		(property "Value" "TLV3502"
 			(at 254 105.41 0)
 			(effects
@@
 			)
 		)
-		(property "Footprint" ""
+		(property "Footprint" "Package_SO:SOIC-8_3.9x4.9mm_P1.27mm"
 			(at 254 113.03 0)
 			(effects
@@
 			)
 		)
-		(property "Datasheet" "http://www.ti.com/lit/ds/symlink/lm393.pdf"
-			(at 254 113.03 0)
+		(property "Datasheet" "https://www.ti.com/lit/gpn/TLV3502"
+			(at 254 106.426 0)
 			(effects
 				(font
@@
 			)
 		)
-		(property "Description" "Low-Power, Low-Offset Voltage, Dual Comparators, DIP-8/SOIC-8/TO-99-8"
-			(at 254 113.03 0)
+		(property "Description" "4.5ns Rail-to-Rail Push-Pull Dual Comparator, SOIC-8"
+			(at 253.492 102.362 0)
 			(effects
 				(font
@@
 			)
 		)
-		(property "Footprint" ""
+		(property "Footprint" "Connector_PinHeader_2.54mm:PinHeader_1x08_P2.54mm_Vertical"
 			(at 241.3 139.7 0)
 			(effects

Commit message: feat: added pcb design
Parts:
- added C6: 100n 100V, Capacitor_SMD:C_0805_2012Metric, symbol Device:C
- D1: value MICROFC-60035-SMT-TR -> MICROFC-60035-SMT; footprint (none) -> muon_sipm:MICROFC-60035-SMT; symbol Device:D_Photo -> muon_sipm:MICROFC-60035-SMT
Connections:
- net GND: now also C6.2
- net SIPM_RAW: now also D1.1 (A); no longer D1.2 (A)
- net VBIAS: now also D1.3 (K), C6.1; no longer D1.1 (K)
- no-connect marks 3 -> 5

Commit message: feat: update detector head to include adc
Parts:
- added C10, C15, C17, C18: 100n, Capacitor_SMD:C_0805_2012Metric, symbol Device:C
- added C11: 2.2p C0G, Capacitor_SMD:C_0805_2012Metric, symbol Device:C
- added C12, C9: 1u, Capacitor_SMD:C_0805_2012Metric, symbol Device:C
- added C13, C7: 10n 100V C0G, Capacitor_SMD:C_0805_2012Metric, symbol Device:C
- added C14: 27p C0G, Capacitor_SMD:C_0805_2012Metric, symbol Device:C
- added C16: 220p C0G, Capacitor_SMD:C_0805_2012Metric, symbol Device:C
- added C8: 1u 50V, Capacitor_SMD:C_1206_3216Metric, symbol Device:C
- added D2: BAS70, Package_TO_SOT_SMD:SOT-23, symbol MuonTelescopeParts:BAS70
- added D3: BAT54S, Package_TO_SOT_SMD:SOT-23, symbol Diode:BAT54S
- added J2: INJECT, Connector_PinHeader_2.54mm:PinHeader_1x02_P2.54mm_Vertical, symbol Connector_Generic:Conn_01x02
- added Q1: BSS138P, Package_TO_SOT_SMD:SOT-23, symbol Transistor_FET:BSS138
- added R10: 4.70k, Resistor_SMD:R_0805_2012Metric, symbol Device:R
- added R11, R8: 1.00k, Resistor_SMD:R_0805_2012Metric, symbol Device:R
- added R12: 499, Resistor_SMD:R_0805_2012Metric, symbol Device:R
- added R13: 82.0, Resistor_SMD:R_0805_2012Metric, symbol Device:R
- added R14, R9: 100, Resistor_SMD:R_0805_2012Metric, symbol Device:R
- added R15: 100k, Resistor_SMD:R_0805_2012Metric, symbol Device:R
- added R16: 2.00k, Resistor_SMD:R_0805_2012Metric, symbol Device:R
- added R17, R18: 0, Resistor_SMD:R_0805_2012Metric, symbol Device:R
- added R19: 330k, Resistor_SMD:R_0805_2012Metric, symbol Device:R
- added TP1: VBIAS, TestPoint:TestPoint_Pad_D2.0mm, symbol Connector:TestPoint
- added TP10: TRIG, TestPoint:TestPoint_Pad_D2.0mm, symbol Connector:TestPoint
- added TP11: PEAK_HOLD, TestPoint:TestPoint_Pad_D2.0mm, symbol Connector:TestPoint
- added TP12: PEAK_OUT, TestPoint:TestPoint_Pad_D2.0mm, symbol Connector:TestPoint
- added TP13: PEAK_RESET, TestPoint:TestPoint_Pad_D2.0mm, symbol Connector:TestPoint
- added TP14, TP15, TP16, TP17, TP18, TP19, TP20: GND_LOOP, MuonTelescopeParts:TestPoint_GroundLoop_P5.00mm_Drill1.0mm, symbol Connector:TestPoint
- added TP2: BIAS_LOCAL, TestPoint:TestPoint_Pad_D2.0mm, symbol Connector:TestPoint
- added TP3: +5V, TestPoint:TestPoint_Pad_D2.0mm, symbol Connector:TestPoint
- added TP4: +3.3V, TestPoint:TestPoint_Pad_D2.0mm, symbol Connector:TestPoint
- added TP5: VBASE, TestPoint:TestPoint_Pad_D2.0mm, symbol Connector:TestPoint
- added TP6: SIPM_RAW, TestPoint:TestPoint_Pad_D2.0mm, symbol Connector:TestPoint
- added TP7: AMP_OUT, TestPoint:TestPoint_Pad_D2.0mm, symbol Connector:TestPoint
- added TP8: VTH, TestPoint:TestPoint_Pad_D2.0mm, symbol Connector:TestPoint
- added TP9: COMP_RAW, TestPoint:TestPoint_Pad_D2.0mm, symbol Connector:TestPoint
- added U3: TPH2502, Package_SO:SOIC-8_3.9x4.9mm_P1.27mm, symbol Amplifier_Operational:LM358
- added U4: TMUX1101, Package_TO_SOT_SMD:SOT-353_SC-70-5, symbol Analog_Switch:TMUX1101DCK
- added U5: SN74LVC1G123, Package_SO:SSOP-8_2.95x2.8mm_P0.65mm, symbol 74xGxx:74LVC1G123
- C3: value 10u -> 4.7u
- J1: value Conn_01x08 -> B10B-XH-A; footprint Connector_PinHeader_2.54mm:PinHeader_1x08_P2.54mm_Vertical -> Connector_JST:JST_XH_B10B-XH-A_1x10_P2.50mm_Vertical; symbol Connector_Generic:Conn_01x08 -> Connector_Generic:Conn_01x10
- RV1: footprint Potentiometer_SMD:Potentiometer_Bourns_3314G_Vertical -> Potentiometer_THT:Potentiometer_Bourns_3296W_Vertical
Connections:
- net +3.3V: now also U2.6 (-), C15.1, D3.2 (K), R10.1, R16.1, TP4.1, U5.3 (~{CLR}), U5.8 (VCC); no longer RV1.1
- net +5V: now also C17.1, C18.1, TP3.1, U3.8 (V+), U4.5 (V_{DD})
- net AMP_OUT: now also C11.2, R8.1, TP7.1, U3.3 (+); no longer U2.3 (+)
- net GND: now also D1.4 (NC), RV1.1, U2.5 (+), C10.2, C12.2, C13.2, C15.2, C16.2, C17.2, C18.2, C7.2, C8.2, C9.2, D3.1 (A), J2.2 (Pin_2), R11.2, R15.2, TP14.1, TP15.1, TP16.1, TP17.1, TP18.1, TP19.1, TP20.1, U3.4 (V-), U4.3 (GND), U5.1 (~{A}), U5.4 (GND); no longer RV1.3
- net SIPM_RAW: now also R12.1, TP6.1
- net TRIG: now also R7.2, TP10.1; no longer R7.1
- net VBASE: now also Q1.2 (S), TP5.1, U4.2
- net VBASE_DIV: now also C10.1, C9.1
- net VBIAS: now also R9.1, TP1.1; no longer D1.3 (K)
- net VTH: now also C13.1, TP8.1
- net AMP_FB: now reaches R5.2, R6.1, U1.2 (-)
- net AMP_FB: now also C11.1
- net COMP_RAW: now reaches U2.1
- net COMP_RAW: now also R18.1, R19.1, TP9.1, U5.2 (B); no longer R7.2
- new net: C12.1, R10.2, R11.1, RV1.3
- new net: R17.2, R18.2, R7.1
- new net: R17.1, U5.5 (Q)
- new net: R13.1, U3.1
- new net: D2.1 (A), R13.2
- new net: C14.2, R16.2, U5.7 (RCext)
- new net: C14.1, U5.6 (Cext)
- new net BIAS_LOCAL: C7.1, C8.1, D1.3 (K), R9.2, TP2.1
- new net COMP_IN: D3.3 (COM), R19.2, R8.2, U2.3 (+)
- new net INJECT: J2.1 (Pin_1), R12.2
- new net PEAK_GUARD: R14.1, U3.6 (-), U3.7
- new net PEAK_HOLD: C16.1, D2.3 (K), Q1.3 (D), TP11.1, U3.2 (-), U3.5 (+), U4.1
- new net PEAK_OUT: J1.9 (Pin_9), R14.2, TP12.1
- new net PEAK_RESET: J1.10 (Pin_10), Q1.1 (G), R15.1, TP13.1, U4.4
- no-connect marks 5 -> 2
Other:
- note added: "BASELINE FILTER de-noises the 50 mV divider. Caps direct noise to ground. C9 covers 70 Hz to few MHz. C10 covers after few MHz."
- note added: "C11 sits across R5 (12.4k): U1A stability option."
- note added: "Fit R17 (stretched, default) OR R18 (direct) - never both. R16 + C14 set the pulse width. R7 damps the cable."
- note added: "J2 pin 1 = INJECT, pin 2 = GND (mark both on both PCB sides)."
- note added: "OPTIONAL PARTS - DNP (not fitted unless bench tests need them)"
- note added: "PEAK CAPTURE & HOLD - U3 holds the biggest pulse since the last reset, for the ADC"
- note added: "Pads: 2.0 mm exposed copper (component side). Ground loops: two 1.0 mm holes, 5.0 mm apart, with a bent wire. Put each loop within 5 mm of the pad in the same row."
- note added: "R10/R11 limit VTH to 0-0.53 V so the 10-turn pot (3296W) gives fine steps. Pot pin 3 = divider, pin 1 = GND, so turning clockwise raises VTH."
- note added: "R13 (R_CHG) and C16 (C_HOLD) are bench-tuned: start at 82.0 ohm / 220 pF C0G. Reset: fit Q1 (BSS138P, default) OR U4 (TMUX1101, precision) - never both. PCB: keep PEAK_HOLD tiny and ring it with a PEAK_GUARD trace."
- note added: "R19 adds ~10 mV of hysteresis. D3 clamps COMP_IN between GND and 3.3 V."
- note added: "SIGNAL INJECTION - test the amplifier without a SiPM"
- note added: "SiPM BIAS FILTER C8-R9 form low-pass filter to let steady 27V through. C7 supplies fast current source to SiPM. Place C7 and C8 right beside the SiPM on the PCB."
- note added: "TEST POINTS - probe pads + ground loops for the scope clip"
- note added: "THRESHOLD - sets the comparator trip level VTH"
- note added: "TRIGGER STRETCHER - U5 turns each comparator edge into a ~200 ns pulse"
- note added: "U1B's job is to produce a constant tiny voltage VBASE (50 mV) that U1A uses as baseline. U1A can't use 0 as baseline because the AC coupling from C1 forces a 0 average V so (+) pulses will force (-) pulses after, and when (-) V are fed into op-amps, they need time to recover & ruin signal integrity. We're using a V divider to get that tiny V, but it's output fluctuates with load & comes with high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"
- note added: "U1C sets max & min of U1A output --------------- 5V leaves room for massive high V events from SiPM."
- note added: "cable has its own impedance. R7 smooths out overall V output --------- The target is R7 + driver output impedance ≈ cable impedance"
- note removed: "U1B's job is to produce a constant tiny voltage VBASE (50 mV) that U1A uses as baseline. U1A can't use 0 as baseline because the AC coupling from C1 forces a 0 average voltage so positive pulses will result in negative pulses afterwards, and when negative vultages are fed into op-amps, they need time to recover & ruin signal integrity. We're using a voltage divider to get that tiny voltage, but i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"
- note removed: "U1C dictates max & min of U1A output --------------- We want 5V to leave room for massive high V events coming from the SiPM."
- note removed: "cable has its own impedance. R7 smooths out overall V output --------- The target is R7 + comparator output impedance ≈ cable impedance"
- moved on the sheet: C1, C2, C3, C4, C5, C6, D1, R1, R2, R3, R4, R5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

Commit message: feat: power board
Other:
- note added: "Decoupling C: Connected in parallel between the power pins and ground (near an IC) to stabilize voltage and shunt high-freq noise -------- The 100n is small and fast - good at high freq. The 10u holds more charge but is slower - good for larger, slower load changes. Together they cover a wider band than either alone. -------- The rule is: capacitor as close to the IC's supply pins as you can phys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"
- note added: "OPTIONAL PARTS - DNP (not fitted unless bench tests need them) R19 adds ~10 mV of hysteresis. D3 clamps COMP_IN between GND and 3.3 V. C11 sits across R5 (12.4k): U1A stability option."
- note added: "PEAK CAPTURE & HOLD - U3 holds the biggest pulse since the last reset, for the ADC U3A setup is voltage follower, but D2 ensures no backflow from C16. FPGA controls PEAK_RESET, which controls the Q1 switch to drain/fill C16. R13 (R_CHG) and C16 (C_HOLD) are bench-tuned: start at 82.0 ohm / 220 pF C0G. Reset: fit Q1 (BSS138P, default) OR U4 (TMUX1101, precision) - never both. PCB: keep PEAK_HOLD t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"
- note added: "THRESHOLD - sets the comparator trip level VTH RV1: potentiometer; below V_set, output is 0V, above, output is 3.3V C12 & C13 shunt noise to ground. R10/R11 limit VTH to 0-0.53 V so the 10-turn pot (3296W) gives fine steps."
- note added: "TRIGGER STRETCHER - U5 turns each comparator edge into a ~200 ns pulse U5A is a one-shot chip; A rise on makes Q go high for a `fixed time` C14-R16 sets this `fixed time`; larger R or C means longer C15 provides fast current source to Q"
- note removed: "C11 sits across R5 (12.4k): U1A stability option."
- note removed: "Decoupling C: Connected in parallel between the power pins and ground (near an IC) to stabilize voltage and shunt high-freq noise -------- Why two values per rail: a real C stops behaving like a C above its self-resonant freq, where its own package inductance takes over. -------- The 100n is small and fast - good at high freq. The 10u holds more charge but is slower - good for larger, slower load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"
- note removed: "J2 pin 1 = INJECT, pin 2 = GND (mark both on both PCB sides)."
- note removed: "OPTIONAL PARTS - DNP (not fitted unless bench tests need them)"
- note removed: "PEAK CAPTURE & HOLD - U3 holds the biggest pulse since the last reset, for the ADC"
- note removed: "R10/R11 limit VTH to 0-0.53 V so the 10-turn pot (3296W) gives fine steps. Pot pin 3 = divider, pin 1 = GND, so turning clockwise raises VTH."
- note removed: "R13 (R_CHG) and C16 (C_HOLD) are bench-tuned: start at 82.0 ohm / 220 pF C0G. Reset: fit Q1 (BSS138P, default) OR U4 (TMUX1101, precision) - never both. PCB: keep PEAK_HOLD tiny and ring it with a PEAK_GUARD trace."
- note removed: "R19 adds ~10 mV of hysteresis. D3 clamps COMP_IN between GND and 3.3 V."
- note removed: "RV1: potentiometer Below V_set, output is 0V; above, output is 3.3 V --------- set at ~100 mV"
- note removed: "THRESHOLD - sets the comparator trip level VTH"
- note removed: "TRIGGER STRETCHER - U5 turns each comparator edge into a ~200 ns pulse"
- moved on the sheet: C11, C14, C15, C16, C17, C18, C2, C3, C4, D2, D3, J1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
