File: hardware/muon_detector_head/muon_detector_head.kicad_sch (KiCad schematic)
At the start: 69 parts, among them J1 B10B-XH-A, J2 INJECT, Q1 BSS138P, U1 TPH2502, U2 TLV3502, U3 TPH2502, U4 TMUX1101, U5 SN74LVC1G123

Commit message: test: fix validation findings on both boards; review decisions still open
Both boards now pass make check with no blocking findings, but three
layout decisions still need approval before any fabrication release.
See hardware/muon_detector_head/README.md.

- Makefile: run the checker with KiCad's bundled Python on macOS.
- Head: exact manufacturer part values; moved C2, C15, C17 and rebuilt the
  peak-hold corner (R13, D2, C16, Q1, U4, TP11, TP19, R14, C18) to meet the
  proximity checks; added the AMP_OUT/R13 clearance rule.
- Power: added the 1.6 mm / 35 um stackup; moved C4, C6, C12 and the boost
  loop parts (L1, D2, C7, C8, C5, R2-R4) closer and rerouted.
- Relaxed four ground-return limits that are geometrically unreachable.
- Regenerated Gerbers under each fab/ folder (not a reviewed release).

Co-Authored-By: Claude Opus 5 <noreply@anthropic.com>
Parts:
- D1: value MICROFC-60035-SMT -> MICROFC-60035-SMT-TR
- D2: value BAS70 -> BAS70,215
- Q1: value BSS138P -> BSS138P,215
- U1, U3: value TPH2502 -> TPH2502-SR
- U2: value TLV3502 -> TLV3502AIDR
- U4: value TMUX1101 -> TMUX1101DCKR
- U5: value SN74LVC1G123 -> SN74LVC1G123DCTR
Changed lines of the file:
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@@
 			)
 		)
-		(property "Value" "TPH2502"
+		(property "Value" "TPH2502-SR"
 			(at 236.22 113.0299 0)
 			(effects
@@
 			)
 		)
-		(property "Value" "BSS138P"
+		(property "Value" "BSS138P,215"
 			(at 189.23 261.62 0)
 			(effects
@@
 			)
 		)
-		(property "Value" "TLV3502"
+		(property "Value" "TLV3502AIDR"
 			(at 242.57 166.3699 0)
 			(effects
@@
 			)
 		)
-		(property "Value" "TPH2502"
+		(property "Value" "TPH2502-SR"
 			(at 193.04 69.85 0)
 			(effects
@@
 			)
 		)
-		(property "Value" "TPH2502"
+		(property "Value" "TPH2502-SR"
 			(at 125.73 232.41 0)
 			(effects
@@
 			)
 		)
-		(property "Value" "TPH2502"
+		(property "Value" "TPH2502-SR"
 			(at 261.874 261.62 0)
 			(effects
@@
 			)
 		)
-		(property "Value" "MICROFC-60035-SMT"
+		(property "Value" "MICROFC-60035-SMT-TR"
 			(at 22.606 64.516 0)
 			(effects
@@
 			)
 		)
-		(property "Value" "TLV3502"
+		(property "Value" "TLV3502AIDR"
 			(at 252.73 72.39 0)
 			(effects
@@
 			)
 		)
-		(property "Value" "SN74LVC1G123"
+		(property "Value" "SN74LVC1G123DCTR"
 			(at 309.88 152.4 0)
 			(effects
@@
 			)
 		)
-		(property "Value" "SN74LVC1G123"
+		(property "Value" "SN74LVC1G123DCTR"
 			(at 331.47 123.19 0)
 			(effects
@@
 			)
 		)
-		(property "Value" "TMUX1101"
+		(property "Value" "TMUX1101DCKR"
 			(at 219.71 256.54 0)
 			(effects
@@
 			)
 		)
-		(property "Value" "BAS70"
+		(property "Value" "BAS70,215"
 			(at 153.67 236.22 0)
 			(effects
@@
 			)
 		)
-		(property "Value" "TPH2502"
+		(property "Value" "TPH2502-SR"
 			(at 222.25 234.95 0)
 			(effects
@@
 			)
 		)
-		(property "Value" "TPH2502"
+		(property "Value" "TPH2502-SR"
 			(at 147.32 110.49 0)
 			(effects
@@
 			)
 		)
-		(property "Value" "TLV3502"
+		(property "Value" "TLV3502AIDR"
 			(at 254 180.34 0)
 			(effects
