File: hardware/muon_detector_head/muon_detector_head.kicad_pcb (KiCad board)
At the start: 2 copper layers, 70 x 70 mm, 73 parts, among them J1 B10B-XH-A, J2 INJECT, Q1 BSS138P, U1 TPH2502, U2 TLV3502, U3 TPH2502, U4 TMUX1101, U5 SN74LVC1G123

Commit message: test: fix validation findings on both boards; review decisions still open
Both boards now pass make check with no blocking findings, but three
layout decisions still need approval before any fabrication release.
See hardware/muon_detector_head/README.md.

- Makefile: run the checker with KiCad's bundled Python on macOS.
- Head: exact manufacturer part values; moved C2, C15, C17 and rebuilt the
  peak-hold corner (R13, D2, C16, Q1, U4, TP11, TP19, R14, C18) to meet the
  proximity checks; added the AMP_OUT/R13 clearance rule.
- Power: added the 1.6 mm / 35 um stackup; moved C4, C6, C12 and the boost
  loop parts (L1, D2, C7, C8, C5, R2-R4) closer and rerouted.
- Relaxed four ground-return limits that are geometrically unreachable.
- Regenerated Gerbers under each fab/ folder (not a reviewed release).

Co-Authored-By: Claude Opus 5 <noreply@anthropic.com>
Parts:
- D1: value MICROFC-60035-SMT -> MICROFC-60035-SMT-TR
- D2: value BAS70 -> BAS70,215
- Q1: value BSS138P -> BSS138P,215
- U1, U3: value TPH2502 -> TPH2502-SR
- U2: value TLV3502 -> TLV3502AIDR
- U4: value TMUX1101 -> TMUX1101DCKR
- U5: value SN74LVC1G123 -> SN74LVC1G123DCTR
- moved C18 26.1 mm to (27.4, 45.6), turned to -90 degrees
- moved TP19 20.4 mm to (19.9, 53.8), turned to 90 degrees
- moved U4 20.2 mm to (23.3, 45.6), turned to 0 degrees
- moved Q1 14.2 mm to (22.1, 42.5), turned to 180 degrees
- moved TP11 13.9 mm to (19.9, 45.8)
- moved D2 7.08 mm to (15.8, 42.6), turned to 0 degrees
- moved C16 6.53 mm to (19.1, 42.5)
- moved R13 6.07 mm to (14.2, 38.6), turned to -90 degrees
- moved C2 5.89 mm to (31.2, 19.0), turned to -90 degrees
- moved C17 4.81 mm to (19.0, 34.2), turned to 180 degrees
- moved R14 2.20 mm to (26.6, 38.6)
- moved C15 1.64 mm to (57.8, 29.3), turned to 90 degrees
Routing:
- net +5V: track 94.1 -> 68.5 mm, vias 7 -> 8
- net /PEAK_RESET: track 95.4 -> 73.3 mm
- net /PEAK_GUARD: track 29.5 -> 10.9 mm
- net /PEAK_HOLD: track 26.0 -> 17.9 mm
- net /VBASE: track 64.9 -> 61.5 mm, vias 6 -> 7
- net +3.3V: track 109.9 -> 107.3 mm
- net /AMP_OUT: track 59.5 -> 57.0 mm, vias 0 -> 2
- net GND: track 33.2 -> 31.3 mm, vias 27 -> 29
- net /SIPM_RAW: track 32.3 -> 30.7 mm
- net /PEAK_OUT: track 57.6 -> 56.3 mm, vias 4 -> 2
- net /COMP_RAW: track 33.3 -> 32.2 mm
- net Net-(U5A-Q): track 2.58 -> 1.77 mm
- net Net-(U5A-Cext): track 3.58 -> 2.78 mm
- net Net-(U5A-RCext): track 6.03 -> 5.27 mm
