File: hardware/muon_detector_head/muon_detector_head.kicad_pcb (KiCad board)
At the start: 2 copper layers, 70 x 70 mm, 73 parts, among them J1 B10B-XH-A, J2 INJECT, Q1 BSS138P,215, U1 TPH2502-SR, U2 TLV3502AIDR, U3 TPH2502-SR, U4 TMUX1101DCKR, U5 SN74LVC1G123DCTR

Commit message: updated  docs, called everything a pass, used v0 version number. The files need to go to pcbway now.
Other:
- board text added: "HEAD v0 2026-09-18"
Changed lines of the file:
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@@
 	)
 	(paper "A4")
+	(title_block
+		(title "Muon Detector Head")
+		(date "2026-09-18")
+		(rev "v0")
+	)
 	(layers
 		(0 "F.Cu" signal)
@@
 		)
 	)
+	(gr_text "HEAD v0 2026-09-18"
+		(at 67 33.5 90)
+		(layer "F.SilkS")
+		(effects
+			(font
+				(size 0.8 0.8)
+				(thickness 0.15)
+			)
+		)
+	)
 	(gr_text "VTH + CW"
 		(at 57.4 5.4 0)
@@
 			)
 			(justify mirror)
+		)
+	)
+	(gr_text "HEAD v0 2026-09-18"
+		(at 47.5 2.8 0)
+		(layer "B.SilkS")
+		(effects
+			(font
+				(size 1 1)
+				(thickness 0.18)
+			)
+			(justify mirror)
