File: hardware/power_interface/power_interface.kicad_pcb (KiCad board)
At the start: 2 copper layers, 96 x 64 mm, 64 parts, among them J1 PJ-102AH, J2 BIAS_EN, J3 B10B-XH-A, J4 B10B-XH-A, J5 TSW-106-08-G-D-RA, U1 TLV75533PDBVR, U2 MAX5026EUT+T, U3 MCP3202-BI/SN

Commit message: test: fix validation findings on both boards; review decisions still open
Both boards now pass make check with no blocking findings, but three
layout decisions still need approval before any fabrication release.
See hardware/muon_detector_head/README.md.

- Makefile: run the checker with KiCad's bundled Python on macOS.
- Head: exact manufacturer part values; moved C2, C15, C17 and rebuilt the
  peak-hold corner (R13, D2, C16, Q1, U4, TP11, TP19, R14, C18) to meet the
  proximity checks; added the AMP_OUT/R13 clearance rule.
- Power: added the 1.6 mm / 35 um stackup; moved C4, C6, C12 and the boost
  loop parts (L1, D2, C7, C8, C5, R2-R4) closer and rerouted.
- Relaxed four ground-return limits that are geometrically unreachable.
- Regenerated Gerbers under each fab/ folder (not a reviewed release).

Co-Authored-By: Claude Opus 5 <noreply@anthropic.com>
Parts:
- moved C12 5.12 mm to (74.3, 43.2), turned to 180 degrees
- moved C4 4.58 mm to (44.5, 38.2), turned to 180 degrees
- moved C6 4.57 mm to (20.0, 19.2), turned to 0 degrees
- moved L1 3.54 mm to (14.4, 25.4)
- moved C8 2.94 mm to (23.8, 26.1), turned to 90 degrees
- moved C7 2.75 mm to (21.4, 26.1), turned to 90 degrees
- moved C5 2.63 mm to (13.6, 18.4), turned to 0 degrees
- moved R2 2.34 mm to (23.1, 22.0), turned to 90 degrees
- moved R3 1.84 mm to (23.1, 18.5)
- moved R4 1.49 mm to (17.2, 17.7)
- moved D2 0.91 mm to (19.3, 25.7), turned to 90 degrees
Routing:
- net GND: track 36.4 -> 285.1 mm, vias 27 -> 37
- net /+3V3_ADC: track 23.5 -> 18.7 mm
- net /LX: track 7.96 -> 3.52 mm
- net Net-(R3-Pad2): track 5.98 -> 7.97 mm
- net /FB: track 10.3 -> 8.69 mm
- net /HV_RAW: track 23.4 -> 22.1 mm
- net /TRIG_B: track 46.4 -> 45.4 mm
- net /SHDN: track 14.0 -> 14.7 mm
- net /+5VA: track 140.8 -> 141.4 mm
